Commit message: Changes in the World

File: sc_gazebo_world/urdf/turtlebot3_waffle_pi.urdf.xacro (robot description, xacro)
@@ -2,5 +2,5 @@
 <robot name="turtlebot3_waffle_pi" xmlns:xacro="http://ros.org/wiki/xacro">
   <xacro:include filename="$(find turtlebot3_description)/urdf/common_properties.xacro"/>
-  <xacro:include filename="$(find turtlebot_follower)/urdf/turtlebot3_waffle_pi.gazebo.xacro"/>
+  <xacro:include filename="$(find sc_gazebo_world)/urdf/turtlebot3_waffle_pi.gazebo.xacro"/>
   <link name="base_footprint"/>
   <joint name="base_joint" type="fixed">

File: sc_gazebo_world/urdf/turtlebot3_waffle_pi_with_marker.urdf.xacro (robot description, xacro)
@@ -207,5 +207,5 @@
       <origin xyz="0 0 0" rpy="0 0 0"/>
       <geometry>
-        <mesh filename="package://turtlebot_follower/meshes/tag36_11_00000_with_border.dae"/>
+        <mesh filename="package://sc_gazebo_world/meshes/tag36_11_00000_with_border.dae"/>
       </geometry>
     </visual>
